File: 02_Schematics_and_boards/Eagle/Mini_VFD_UI_RevA.sch (EAGLE design)
At the start: 80 parts, among them IC1 TCA9534ADWR, IC2 SN74LVC14ADR, IC3 SPX1117M3, M1 DOGL128, Q1 BSS138P, Q2 BSS138P, Q3 BSS138P, Q4 BSS138P, SW1 EC12E_SW, X1 057-020-1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

Commit message: Edited Documentation
Other:
- note added: "Aux. UART Header"
- note removed: "EEPROM"
- note removed: "STM32 Microcontroller"
Changed lines of the file:
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@@
 <part name="+3V19" library="supply_MICHAEL" deviceset="+3.3V" device=""/>
 <part name="R28" library="rcl_MICHAEL" deviceset="R-EU_" device="R0603" package3d_urn="urn:adsk.eagle:package:23555/3" value="10k"/>
-<part name="X2" library="Connectors" deviceset="DF3E-4P-2V" device="" package3d_urn="urn:adsk.eagle:package:39324394/2" value="DF3E-4P-2V(51)"/>
+<part name="X2" library="Connectors" deviceset="DF3E-4P-2V" device="" package3d_urn="urn:adsk.eagle:package:39324394/2" value="DF3E-4P-2V(51)">
+<variant name="Assembly_1" populate="no"/>
+</part>
 <part name="+3V20" library="supply_MICHAEL" deviceset="+3.3V" device=""/>
 <part name="GND33" library="supply1" library_urn="urn:adsk.eagle:library:371" deviceset="GND" device=""/>
@@
 <wire x1="264.16" y1="12.7" x2="12.7" y2="12.7" width="0.254" layer="97"/>
 <wire x1="12.7" y1="12.7" x2="12.7" y2="248.92" width="0.254" layer="97"/>
-<text x="15.24" y="243.84" size="2.54" layer="97" ratio="12">STM32 Microcontroller</text>
+<text x="15.24" y="243.84" size="2.54" layer="97" ratio="12">LCD Display</text>
 <wire x1="271.78" y1="104.14" x2="375.92" y2="104.14" width="0.254" layer="97"/>
 <wire x1="375.92" y1="104.14" x2="375.92" y2="33.02" width="0.254" layer="97"/>
@@
 <wire x1="375.92" y1="111.76" x2="271.78" y2="111.76" width="0.254" layer="97"/>
 <wire x1="271.78" y1="111.76" x2="271.78" y2="170.18" width="0.254" layer="97"/>
-<text x="274.32" y="165.1" size="2.54" layer="97" ratio="12">EEPROM</text>
+<text x="274.32" y="165.1" size="2.54" layer="97" ratio="12">Aux. UART Header</text>
 </plain>
 <instances>
